File: MakerBot.sch (EAGLE design)
At the start: 52 parts, among them U10 MCP4018, U11 MCP4018, U8 MCP4018, U9 MCP4018

Commit message: Designed! Routed! Time to build!
Parts:
- removed U10, U11, U8, U9: MCP4018, MakerBot:MCP4018
- added INTERFACE, INTERFACE1, INTERFACE2, INTERFACE3: (no value), con-ml:ML6
- added POWER: 9090-4V, con-thomas-betts:9090-4V
- C10, C11, C12, C13: device adafruit:C-US -> adafruit:C-US050-075X075
- R10, R103, R104, R20, R21, R22, R23, R34, R35, R39, R40, R5, R6, R7, R8, R9: device SparkFun:RESISTOR -> SparkFun:RESISTORPTH1
Connections:
- removed net A-AXIS-POT: R106.2
- removed net N$112: R35.1, U9.A
- removed net N$126: R36.1, U10.A
- removed net N$176: R37.1, U11.A
- removed net N$356: R103.1, U8.SDA
- removed net N$357: R104.1, U9.SDA
- removed net N$359: R105.1, U10.SDA
- removed net N$361: R106.1, U11.SDA
- removed net N$98: R34.1, U8.A
- removed net POTS-SCL: U10.SCL, U11.SCL, U8.SCL, U9.SCL
- removed net X-AXIS-POT: R103.2
- removed net Y-AXIS-POT: R104.2
- removed net Z-AXIS-POT: R105.2
- new net N$1: R15.1, R27.2
- new net N$2: R14.1, R26.2
- new net RESET: INTERFACE.6, INTERFACE1.6, INTERFACE2.6, INTERFACE3.6
- net +24V: now also POWER.4
- net 5V: now also POWER.1; no longer U10.VDD, U11.VDD, U8.VDD, U9.VDD
- net A-AXIS-DIR: now also INTERFACE3.4
- net A-AXIS-EN: now also INTERFACE3.5
- net A-AXIS-STEP: now also INTERFACE3.3
- net GND: now also INTERFACE.1, INTERFACE.2, INTERFACE1.1, INTERFACE1.2, INTERFACE2.1, INTERFACE2.2, INTERFACE3.1, INTERFACE3.2, POWER.2, POWER.3; no longer U10.VSS, U11.VSS, U8.VSS, U9.VSS
- net N$111: no longer U9.W
- net N$124: no longer U10.W
- net N$173: no longer U11.W
- net N$177: no longer R15.1, R27.2
- net N$188: no longer R14.1, R26.2
- net N$96: no longer U8.W
- net X-AXIS-DIR: now also INTERFACE.4
- net X-AXIS-EN: now also INTERFACE.5
- net X-AXIS-STEP: now also INTERFACE.3
- net Y-AXIS-DIR: now also INTERFACE1.4
- net Y-AXIS-EN: now also INTERFACE1.5
- net Y-AXIS-STEP: now also INTERFACE1.3
- net Z-AXIS-DIR: now also INTERFACE2.4
- net Z-AXIS-EN: now also INTERFACE2.5
- net Z-AXIS-STEP: now also INTERFACE2.3
